File: KiCad/Coche teledirigido.kicad_sch (KiCad schematic)
At the start: 55 parts, among them J1 USB_A_5A, J10 Conn_M1_M, J11 Conn_01x04_Male, J12 Conn_Servo1_F, J13 Conn_Servo2_F, J14 Conn_Servo3_F, J15 Conn_M1_F, J16 HC-05 Bluetooth, J2 USB_A_10A, J3 USB_A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

Commit message: Actualizar
Parts:
- removed U1: 74164, symbol 74xx_IEEE:74164
- added U?: 74HC595, symbol 74xx:74HC595
Connections:
- net +5v (10.000mA): now also U?.10 (~{SRCLR}), U?.16 (VCC)
- net Earth: now also U?.13 (~{OE}), U?.8 (GND)
- net INT_IZQ: now also U?.7 (QH)
- net LUZ_CRU: now also U?.3 (QD)
- net PWM3: now also J8.1 (Pin_1); no longer J7.1 (Pin_1)
- net PWM5: now also J9.1 (Pin_1); no longer J8.1 (Pin_1)
- net PWM6: now also J7.1 (Pin_1); no longer J9.1 (Pin_1)
- net SIR_AZU: now also U?.4 (QE)
- net SIR_ROJ: now also U?.5 (QF)
- net CK16 renamed DS16
- net DS16: now also U?.14 (SER)
- net DD14 renamed STCP14
- net STCP14: now also U?.12 (RCLK)
- net RS10 renamed SHCP
- new net SHCP10: U?.11 (SRCLK)
